File: Electronics/lcdboard.brd (EAGLE design)
At the start: 100 x 57 mm, 19 parts, among them IC1 MCP23017SP, IC3 1117-33, IC5 4050N, U2 USD-SOCKETUSD

Commit message: update
Other:
- board text added: "1K"
Changed lines of the file:
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@@
 <wire x1="90" y1="-15" x2="90" y2="-5" width="0.1524" layer="20"/>
 <text x="13.1" y="25.9" size="0.8128" layer="21" ratio="15" rot="R90">10K</text>
-<text x="78" y="24.8" size="0.8128" layer="21" ratio="15" rot="R90">10K</text>
+<text x="78" y="24.8" size="0.8128" layer="21" ratio="15" rot="R90">1K</text>
 <text x="80.4" y="24.9" size="0.8128" layer="21" ratio="15" rot="R90">10K</text>
 <text x="83" y="24.8" size="0.8128" layer="21" ratio="15" rot="R90">10K</text>
