File: Electronics/miniprinter-sanguinololu-longboard.brd (EAGLE design)
At the start: 250 x 40 mm, 73 parts, among them IC100 FT232RL, IC2 ATMEGA644-20PU, J1 USB, P1 POLOLU-X, P2 POLOLU-Y, P3 POLOLU-Z, P4 POLOLU-E, Q1 RFP30N06LE, Q2 RFP30N06LE, Q4 RFP30N06LE, X1 MSTBA2, X2 MSTBA2, X3 MSTBA2, X4 MSTBA2

Commit message: update
Parts:
- R1: value 10k -> 100k
Changed lines of the file:
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@@
 <attribute name="VALUE" x="196.298" y="-19.002" size="1.27" layer="27" ratio="10"/>
 </element>
-<element name="R1" library="SparkFun" package="AXIAL-0.3" value="10k" x="199.6" y="-18.7" smashed="yes">
+<element name="R1" library="SparkFun" package="AXIAL-0.3" value="100k" x="199.6" y="-18.7" smashed="yes">
 <attribute name="NAME" x="197.06" y="-17.43" size="0.4064" layer="25"/>
 <attribute name="VALUE" x="197.568" y="-19.208" size="0.8128" layer="21" ratio="15"/>
