File: V3 Controller/MiniPrinterController.brd (EAGLE design)
At the start: 100 x 100 mm, 153 parts, among them IC9 XL1509-5.0E1, Q1 IRLR024, Q2 IRLR024, Q22 IRLR024, SW1 Legion SS21BBINPD Switch

Commit message: update
Parts:
- removed J5: (no value), SparkFun-Connectors:2X5-SHROUDED_LOCK
- removed SV1, SV2, SV3, SV4, SV5: (no value), con-lstb:MA04-1
- removed SV6: (no value), con-lstb:MA05-1
- removed SW1: Legion SS21BBINPD Switch, openbuilds-eagle-library:POWER-LEGION-SS21-ROCKER-SWITCH
- removed U$3, U$5: ATQ-FUSE, ATQ Fuse Holder out of 4.3mm pcb terminals:ATQ-FUSE
- removed X-END: Phoenix Pluggable 3.81mm 2 way, jt-con-phoenix-3.81:MC1.5/2-G-3.81
- added ETHERM: Phoenix Pluggable 3.81mm 2 way, jt-con-phoenix-3.81:MC1.5/2-G-3.81
- added J1, J2: (no value), SparkFun-Connectors:2X5-SHROUDED_LOCK
- added JP1: (no value), pinhead:1X12
- added JP3: (no value), pinhead:1X16
- LED6: device adafruit:CHIPLED_0805 -> adafruit:LED3MM
- moved D18 332.1 mm to (87.4, 2.50), flipped to the bottom, turned to 0 degrees
- moved C56 332.1 mm to (87.5, 16.5), flipped to the top, turned to 0 degrees
- moved BEDTH 324.8 mm to (40.0, 0.00)
- moved C4 324.3 mm to (38.5, 12.0), flipped to the bottom
- moved C3 323.9 mm to (39.0, 18.5), flipped to the bottom
- moved R26 323.9 mm to (39.0, 22.0), flipped to the bottom
- moved R27 323.9 mm to (39.0, 15.5), flipped to the bottom
- moved BED 318.5 mm to (27.0, 5.00)
- moved D2 318.1 mm to (27.0, 14.0), flipped to the bottom, turned to 0 degrees
- moved MOS2 315.9 mm to (29.0, 23.0), flipped to the bottom
- moved R24 315.6 mm to (29.0, 38.0), flipped to the bottom, turned to 180 degrees
- moved R25 315.6 mm to (29.0, 35.0), flipped to the bottom
- moved L2 315.3 mm to (96.0, 11.5)
- moved D11 314.5 mm to (87.5, 8.50), flipped to the bottom, turned to 0 degrees
- moved C42 309.2 mm to (87.5, 5.50), flipped to the top
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Connections:
- removed net N$4: BED.2, U$3.TERM2.1, U$3.TERM2.2
- removed net PROBE: J8.9
- removed net V+FUSE: D14.C, SW1.L2, SW1.R2, U$4.TERM2.1, U$4.TERM2.2
- removed net VM-HOTEND: J5.4, J5.5, J5.6, U$5.TERM2.1, U$5.TERM2.2, X-END1.2, X-END2.2, X-END3.2
- removed net X-END-C1: J7.9
- removed net Y-ENDSTOP-C1: J6.9
- removed net Z-ENDSTOP-C1: Z-CONN1.9
- new net N$40: JP1.9
- new net SPARE1: J2.10
- new net SPARE2: J2.9
- new net _E-ENDSTOP-C1: J7.9, JP3.1
- new net _X-ENDSTOP-C1: JP3.4, Z-CONN1.9
- new net _Y-ENDSTOP-C1: J6.9, JP3.3
- new net _Z-ENDSTOP-C1: J8.9, JP3.2
- net 5VREG: now also JP1.11
- net AGND: now also BEDTH.1, ETHERM.1, J1.9, JP1.5; no longer BEDTH.2, J5.9, SV5.1
- net AVCC: now also JP1.6; no longer SV5.2
- net BED: now also JP1.1; no longer SV6.2
- net E-FAN: now also JP1.3; no longer SV6.3
- net E-FAN-NEG: now also J2.1, J2.2; no longer J5.7
- net EDIR: now also JP3.7; no longer SV4.4
- net EENABLE: now also JP3.5; no longer SV4.2
- net ESTEP: now also JP3.6; no longer SV4.3
- net GND: now also JP1.12; no longer SV1.1, SV2.1, SV3.1, SV4.1, SV6.1
- net HOTEND: now also JP1.2; no longer SV6.5
- net HOTEND-NEG1: now also J1.1, J1.2, J1.3, J1.4; no longer J5.1, J5.2, J5.3
- net N$16: now also LED6.K; no longer LED6.C
- net PART-FAN: now also JP1.4; no longer SV6.4
- net PART-FAN-NEG: now also J2.5, J2.6; no longer J5.8
- net TH1_HOTEND: now also ETHERM.2, J1.10, JP1.8; no longer J5.10, SV5.3
- net TH2_BED: now also BEDTH.2, JP1.7; no longer BEDTH.1, SV5.4
- net VM: now also BED.2, D14.C, J1.5, J1.6, J1.7, J1.8, J2.3, J2.4, J2.7, J2.8, JP1.10, U$4.TERM2.1, U$4.TERM2.2, X-END1.2, X-END2.2, X-END3.2; no longer SW1.L1, SW1.R1, U$3.TERM1.1, U$3.TERM1.2, U$5.TERM1.1, U$5.TERM1.2
- net XDIR: now also JP3.16; no longer SV1.4
- net XENABLE: now also JP3.14; no longer SV1.2
- net XSTEP: now also JP3.15; no longer SV1.3
- net YDIR: now also JP3.13; no longer SV2.4
- net YENABLE: now also JP3.11; no longer SV2.2
- net YSTEP: now also JP3.12; no longer SV2.3
- net ZDIR: now also JP3.10; no longer SV3.4
- net ZENABLE: now also JP3.8; no longer SV3.2
- net ZSTEP: now also JP3.9; no longer SV3.3
Routing:
- net AGND: track 0.00 -> 118.6 mm, vias 0 -> 2
- net TH1_HOTEND: track 0.00 -> 106.7 mm, vias 0 -> 2
- net TH2_BED: track 0.00 -> 98.8 mm, vias 0 -> 1
- net XENABLE: track 18.8 -> 116.1 mm
- net XSTEP: track 18.8 -> 114.6 mm
- net XDIR: track 15.1 -> 109.4 mm
- net AVCC: track 0.00 -> 89.8 mm, vias 0 -> 1
- net YENABLE: track 19.6 -> 101.4 mm
- net _X-ENDSTOP-C1: track 0.00 -> 80.9 mm
- net YSTEP: track 18.9 -> 99.3 mm
- net YDIR: track 15.5 -> 94.1 mm
- net BED: track 0.00 -> 74.8 mm, vias 0 -> 1
- net ZENABLE: track 19.2 -> 85.6 mm
- net ZSTEP: track 19.0 -> 84.0 mm
- net ZDIR: track 15.1 -> 78.5 mm
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- added copper zone on layer 1, net 5VREG
- added copper zone on layer 16, net 5VREG
- added copper zone on layer 16, net AGND
- added copper zone on layer 16, net BED-NEG1
- added copper zone on layer 16, net E-FAN-NEG
- added copper zone on layer 16, net GND
- added copper zone on layer 16, net HOTEND-NEG1
- added copper zone on layer 16, net N$1
- added copper zone on layer 16, net N$26
- added copper zone on layer 16, net PART-FAN-NEG
- added copper zone on layer 16, net TH1_HOTEND
- added copper zone on layer 16, net V+PSU
- removed copper zone on layer 1, net N$26
- removed copper zone on layer 1, net VM
Other:
- board size 100 x 100 mm -> 210 x 100 mm
- board text added: "-"
- board text added: "5V-REG"
- board text added: "A-GND"
- board text added: "A-VCC"
- board text added: "BED"
- board text added: "BEDTH"
- board text added: "E-DIR"
- board text added: "E-EN"
- board text added: "E-END"
- board text added: "E-FAN"
- board text added: "E-FAN+"
- board text added: "E-FAN-"
- board text added: "E-STP"
- board text added: "GND"
- board text added: "H-THER"
- board text added: "HOTEND+"
- board text added: "HOTEND-"
- board text added: "PART-FAN"
- board text added: "PART-FAN+"
- board text added: "PART-FAN-"
- board text added: "SPARE"
- board text added: "TERMISTOR"
- board text added: "TH1-HOTEND"
- board text added: "TH2-BED"
- board text added: "V-IN"
- board text added: "VM"
- board text added: "X-DIR"
- board text added: "X-EN"
- board text added: "X-END"
- board text added: "X-STP"
- board text added: "Y-DIR"
- board text added: "Y-EN"
- board text added: "Y-END"
- board text added: "Y-STP"
- board text added: "Z-DIR"
- board text added: "Z-EN"
- board text added: "Z-END"
- board text added: "Z-STP"
- board text removed: "E-AXIS"
- board text removed: "EXT FAN"
- board text removed: "PART FAN"
- board text removed: "X-AXIS"
- board text removed: "Y-AXIS"
- board text removed: "Z-AXIS"

Commit message: update
Parts:
- added C14, C31, C36: 22p, SmartPrj:C0603-ROUND
- added C28, C29, C5, C6, C7, C8: 100n, SmartPrj:C0603-ROUND
- added C30: 100n, rcl:C0603
- added IC3: ATMEGA2560-16AU, atmel-2005:TQFP100
- added IC5: LM358D, linear:SO08
- added IC6: LP2985-33DBVR, texas:SOT23-DBV
- added ICSP: ICSP, pinhead:2X03
- added JP2: (no value), pinhead:1X16
- added JP4: (no value), pinhead:1X12
- added JP5, JP6: (no value), pinhead:1X01
- added L: YELLOW, led:CHIP-LED0805
- added ON: GREEN, led:CHIP-LED0805
- added Q3: 16MHz, special:QS
- added R54: 27R, SmartPrj:R0603-ROUND
- added R55, R60, R68, R69: 1k, rcl:R0603
- added R61, R64, R65, R66, R67: 10k, rcl:R0603
- added RESET: TS42, st-mod v1.4:TS42
- added SJ10, SJ11, SJ12, SJ13, SJ14, SJ15, SJ16, SJ17, SJ18, SJ19, SJ20, SJ21, SJ22, SJ23, SJ24, SJ25, SJ26, SJ27, SJ28, SJ29, SJ30, SJ31, SJ32, SJ33, SJ34, SJ35, SJ36, SJ9: (no value), jumper:SJ
- added T2: FDN340P, zetex:SOT-23
Connections:
- removed net N$40: JP1.9
- new net +3V3: C28.2, IC5.6, IC6.5
- new net +5V: C30.2, C6.1, C7.1, C8.1, IC3.10, IC3.100, IC3.31, IC3.61, IC3.80, IC5.8, IC6.1, IC6.3, ICSP.2, JP6.1, R60.1, R61.2, R64.2, R65.2, T2.2
- new net 5-GND: RESET.5
- new net 5VREG_CONTROL: JP4.11, SJ35.1
- new net AGND_CONTROL: JP4.5, SJ29.1
- new net AREF: C5.1, IC3.98
- new net AVCC_CONTROL: JP4.6, SJ30.1
- new net BED_CONTROL: JP4.1, SJ25.1
- new net CMP: C29.2, IC5.5, R66.1, R67.2
- new net D0: IC3.2, R68.2
- new net D1: IC3.3, R69.2
- new net D10: IC3.23, SJ9.2
- new net D11: IC3.24
- new net D12: IC3.25
- new net D13: IC3.26, R55.1
- new net D14/TXD3: IC3.64
- new net D15/RXD3: IC3.63
- new net D16/TXD2: IC3.13
- new net D17/RXD2: IC3.12
- new net D18/TXD1: IC3.46
- new net D19/RXD1: IC3.45
- new net D2: IC3.6, SJ13.2
- new net D20/SDA: IC3.44, R65.1
- new net D21/SCL: IC3.43, R64.1
- new net D22: IC3.78
- new net D23: IC3.77
- new net D24: IC3.76
- new net D25: IC3.75
- new net D26: IC3.74
- new net D27: IC3.73
- new net D28: IC3.72
- new net D29: IC3.71
- new net D3: IC3.7, SJ12.2
- new net D30: IC3.60
- new net D31: IC3.59
- new net D32: IC3.58
- new net D33: IC3.57
- new net D34: IC3.56
- new net D35: IC3.55
- new net D36: IC3.54
- new net D37: IC3.53
- new net D38: IC3.50
- new net D39: IC3.70
- new net D4: IC3.1, SJ15.2
- new net D40: IC3.52
- new net D41: IC3.51
- new net D42: IC3.42
- new net D43: IC3.41
- new net D44: IC3.40
- new net D45: IC3.39
- new net D46: IC3.38
- new net D47: IC3.37
- new net D48: IC3.36
- new net D49: IC3.35
- new net D5: IC3.5, SJ14.2
- new net D50/MISO: IC3.22, ICSP.1
- new net D51/MOSI: IC3.21, ICSP.4
- new net D52/SCK: IC3.20, ICSP.3
- new net D53/SS: IC3.19
- new net D54/ADC0: IC3.97
- new net D55/ADC1: IC3.96, SJ16.2
- new net D56/ADC2: IC3.95, SJ17.2
- new net D57/ADC3: IC3.94, SJ18.2
- new net D58/ADC4: IC3.93, SJ19.2
- new net D59/ADC5: IC3.92, SJ20.2
- new net D60/ADC6: IC3.91, SJ21.2
- new net D61/ADC7: IC3.90, SJ22.2
- new net D62/ADC8: IC3.89, SJ23.2
- new net D63/ADC9: IC3.88, SJ24.2
- new net D64/ADC10: IC3.87, SJ25.2
- new net D65/ADC11: IC3.86, SJ26.2
- new net D66/ADC12: IC3.85, SJ27.2
- new net D67/ADC13: IC3.84, SJ28.2
- new net D68/ADC14: IC3.83, SJ31.2
- new net D69/ADC15: IC3.82, SJ32.2
- new net D8: IC3.17, SJ11.2
- new net D9: IC3.18, SJ10.2
- new net E-FAN_CONTROL: JP4.3, SJ27.1
- new net EDIR_CONTROL: JP2.7, SJ15.1
- new net EENABLE_CONTROL: JP2.5, SJ13.1
- new net ESTEP_CONTROL: JP2.6, SJ14.1
- new net GATE_CMD: IC5.7, T2.3
- new net GND_CONTROL: C14.2, C28.1, C29.1, C30.1, C31.1, C36.1, C5.2, C6.2, C7.2, C8.2, IC3.11, IC3.32, IC3.62, IC3.81, IC3.99, IC5.2, IC5.3, IC5.4, IC6.2, ICSP.6, JP4.12, JP4.9, L.C, ON.C, R67.1, RESET.1, RESET.2, SJ33.1, SJ36.1
- new net HOTEND_CONTROL: JP4.2, SJ26.1
- new net M8RXD: R68.1
- new net M8TXD: R69.1
- new net N$13: ON.A, R60.2
- new net N$14: L.A, R55.2
- new net N$30: SJ35.2
- new net N$31: SJ34.2
- new net N$32: SJ33.2
- new net N$35: SJ30.2
- new net N$36: SJ29.2
- new net N$4: SJ36.2
- new net PART-FAN_CONTROL: JP4.4, SJ28.1
- new net PH3: IC3.15
- new net PH4: IC3.16
- new net RESET: C14.1, IC3.30, ICSP.5, R61.1, RESET.3, RESET.4
- new net TH1_HOTEND_CONTROL: JP4.8, SJ32.1
- new net TH2_BED_CONTROL: JP4.7, SJ31.1
- new net USBVCC: JP5.1, T2.1
- new net VIN: R66.2
- new net VM_CONTROL: JP4.10, SJ34.1
- new net XDIR_CONTROL: JP2.16, SJ24.1
- new net XENABLE_CONTROL: JP2.14, SJ22.1
- new net XSTEP_CONTROL: JP2.15, SJ23.1
- new net XTAL1: C31.2, Q3.2, R54.2
- new net XTAL1R: IC3.34, R54.1
- new net XTAL2: C36.2, IC3.33, Q3.1
- new net YDIR_CONTROL: JP2.13, SJ21.1
- new net YENABLE_CONTROL: JP2.11, SJ19.1
- new net YSTEP_CONTROL: JP2.12, SJ20.1
- new net ZDIR_CONTROL: JP2.10, SJ18.1
- new net ZENABLE_CONTROL: JP2.8, SJ16.1
- new net ZSTEP_CONTROL: JP2.9, SJ17.1
- new net _E-ENDSTOP-C1_CONTROL: JP2.1, SJ9.1
- new net _X-ENDSTOP-C1_CONTROL: JP2.4, SJ12.1
- new net _Y-ENDSTOP-C1_CONTROL: JP2.3, SJ11.1
- new net _Z-ENDSTOP-C1_CONTROL: JP2.2, SJ10.1
- net GND: now also JP1.9
Routing:
- net GND_CONTROL: track 0.00 -> 60.6 mm
- net +5V: track 0.00 -> 40.3 mm, vias 0 -> 2
- net RESET: track 0.00 -> 36.2 mm
- net XTAL2: track 0.00 -> 11.1 mm
- net D52/SCK: track 0.00 -> 8.65 mm
- net D51/MOSI: track 0.00 -> 8.65 mm
- net D20/SDA: track 0.00 -> 8.53 mm
- net XTAL1: track 0.00 -> 8.28 mm
- net D50/MISO: track 0.00 -> 7.10 mm, vias 0 -> 1
- net D21/SCL: track 0.00 -> 6.64 mm
- net D0: track 0.00 -> 6.53 mm
- net D1: track 0.00 -> 6.24 mm
- net N$13: track 0.00 -> 3.08 mm
- net N$14: track 0.00 -> 3.04 mm
- net XDIR_CONTROL: track 0.00 -> 2.58 mm
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Other:
- outline, holes or cut-outs redrawn

Commit message: update
Parts:
- removed IC6: LP2985-33DBVR, texas:SOT23-DBV
- added C43, C45, C49, C50: 0.1uF, SparkFun:0603-CAP
- added C44, C47, C51, C52: 10uF, SparkFun:EIA3216
- added C46: 0.1uF, SmartPrj:C0603-ROUND
- added D15: SS34, dp_devices:DO-214AC
- added D21: RED/GRN BICOLOR 3528 LED, Wurth_Elektronik_Optoelectronics_rev15c:3528
- added IC1: 4050D, 40xx:SO16
- added IC2: 1117-33, v-reg:SOT223
- added J3: USB-C-Socket, SparkFun-Connectors:USB-C-16P
- added R70, R71: 5.1k, SparkFun-Resistors:0603@1
- added R72, R73: 1K, SparkFun:0603-RES
- added U2: USD-SOCKETUSD, SparkFun-Connectors_PETERMICROSDEBAY:USD-SOCKET-PP
- added U6: FT232RLSSOP, SparkFun:SSOP28DB
- moved C8 3.12 mm to (169.4, 57.2)
- moved ICSP 1.98 mm to (167.4, 62.7)
- moved R68 1.98 mm to (173.9, 54.2)
- moved R69 1.98 mm to (172.1, 56.0)
- moved RESET 1.98 mm to (174.1, 69.4)
- moved C7 0.45 mm to (165.1, 39.1)
- turned C31 to 45 degrees
- turned C36 to 225 degrees
Connections:
- removed net N$31: SJ34.2
- removed net N$32: SJ33.2
- removed net USBVCC: JP5.1, T2.1
- removed net VIN: R66.2
- new net 3VUSB: C45.1, U6.17
- new net CC1: J3.A5, R71.2
- new net CC2: J3.B5, R70.2
- new net CS: IC1.2, U2.2
- new net CTS: U6.11
- new net D+1: J3.A6, J3.B6, U6.15
- new net D-1: J3.A7, J3.B7, U6.16
- new net D6: IC3.8
- new net D7: IC3.9
- new net DI: IC1.4, U2.3
- new net DTR: C46.1, U6.2
- new net RTS: U6.3
- new net RXLED: R72.1, U6.22
- new net SC: IC1.6, U2.5
- new net SHLD: J3.SHLD1, J3.SHLD2, J3.SHLD3, J3.SHLD4, J3.SHLD5, J3.SHLD6, J3.SHLD7, J3.SHLD8
- new net TXLED: R73.1, U6.23
- new net VM_L2: R66.2, SJ34.2
- new net V_USB: C43.1, C44.A, D15.2, D21.1, D21.2, J3.VBUS1, J3.VBUS2, JP5.1, U6.20, U6.4
- new net V_USB_AFTERDIODE: D15.1, T2.1
- net +3V3: now also C47.A, C49.1, C50.1, C52.A, IC1.1, IC2.4, U2.4; no longer IC6.5
- net +5V: now also C51.A, IC2.3, SJ35.2; no longer IC6.1, IC6.3
- net D50/MISO: now also U2.7
- net D51/MOSI: now also IC1.5
- net D52/SCK: now also IC1.7
- net D53/SS: now also IC1.3
- net GND_CONTROL: now also C43.2, C44.C, C45.2, C47.C, C49.2, C50.2, C51.C, C52.C, IC1.8, IC2.1, J3.GND, J3.GND2, R70.1, R71.1, SJ33.2, SJ36.2, U2.6, U2.GND1, U2.GND2, U6.18, U6.21, U6.25, U6.26, U6.7; no longer IC6.2
- net M8RXD: now also U6.1
- net M8TXD: now also U6.5
- net N$30: now also D21.3, R73.2; no longer SJ35.2
- net N$4: now also D21.4, R72.2; no longer SJ36.2
- net RESET: now also C46.2
Routing:
- net V_USB: track 0.00 -> 43.8 mm
- net GND_CONTROL: track 60.6 -> 27.2 mm, vias 0 -> 18
- net SC: track 0.00 -> 22.9 mm, vias 0 -> 2
- net +3V3: track 0.00 -> 20.4 mm
- net D50/MISO: track 7.10 -> 27.3 mm, vias 1 -> 3
- net D-1: track 0.00 -> 19.2 mm
- net D+1: track 0.00 -> 19.0 mm
- net CS: track 0.00 -> 16.6 mm, vias 0 -> 2
- net DI: track 0.00 -> 14.5 mm, vias 0 -> 2
- net D10: track 0.00 -> 14.4 mm, vias 0 -> 2
- net D9: track 0.00 -> 11.9 mm
- net D4: track 0.00 -> 11.9 mm, vias 0 -> 2
- net D8: track 0.00 -> 11.6 mm
- net D3: track 0.00 -> 10.7 mm
- net D2: track 0.00 -> 10.5 mm
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
Commit message: update
Parts:
- removed JP1, JP4: (no value), pinhead:1X12
- removed JP2, JP3: (no value), pinhead:1X16
- removed SJ10, SJ11, SJ12, SJ13, SJ14, SJ15, SJ16, SJ17, SJ18, SJ19, SJ20, SJ21, SJ22, SJ23, SJ24, SJ25, SJ26, SJ27, SJ28, SJ29, SJ30, SJ31, SJ32, SJ33, SJ34, SJ35, SJ36, SJ9: (no value), jumper:SJ
- added D16, D17, D19, D20: M4, diode:DO-214AC
- added L1, L3: 39nH, SparkFun:0603
- added R74, R75, R76, R77: 1K, resistor:R0603
- added R78, R79, R80, R81: 10K, resistor:R0603
- added U1: TLP291-4, Toshiba TLP291-4 Optocoupler:SO16_TOS
- moved R67 104.1 mm to (102.0, 12.0), flipped to the bottom
- moved R66 99.9 mm to (104.0, 12.0), flipped to the bottom
- moved IC5 96.7 mm to (102.9, 4.80), flipped to the bottom
- moved C29 95.7 mm to (106.0, 12.0), flipped to the bottom
- moved C28 90.2 mm to (108.0, 12.0), flipped to the bottom, turned to 270 degrees
- moved T2 85.5 mm to (109.0, 6.40), flipped to the bottom
- moved JP6 79.5 mm to (112.0, 8.30), flipped to the bottom
- moved JP5 79.5 mm to (112.0, 5.40), flipped to the bottom
- moved D15 76.1 mm to (110.5, 2.10), flipped to the bottom
- moved U2 74.8 mm to (123.7, 83.8), flipped to the bottom, turned to 180 degrees
- moved C52 72.6 mm to (97.8, 66.1), flipped to the bottom
- moved C51 72.2 mm to (97.8, 52.1), flipped to the bottom
- moved IC2 72.1 mm to (97.8, 59.1), flipped to the bottom
- moved C5 71.6 mm to (99.6, 46.8), flipped to the bottom, turned to 0 degrees
- moved R68 70.3 mm to (103.6, 54.7), flipped to the bottom, turned to 270 degrees
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Connections:
- removed net +5V: C30.2, C51.A, C6.1, C7.1, C8.1, IC2.3, IC3.10, IC3.100, IC3.31, IC3.61, IC3.80, IC5.8, ICSP.2, JP6.1, R60.1, R61.2, R64.2, R65.2, SJ35.2, T2.2
- removed net 5VREG_CONTROL: JP4.11, SJ35.1
- removed net AGND_CONTROL: JP4.5, SJ29.1
- removed net AVCC_CONTROL: JP4.6, SJ30.1
- removed net BED: JP1.1, R24.1
- removed net BED_CONTROL: JP4.1, SJ25.1
- removed net D2: IC3.6, SJ13.2
- removed net D4: IC3.1, SJ15.2
- removed net D5: IC3.5, SJ14.2
- removed net D55/ADC1: IC3.96, SJ16.2
- removed net D56/ADC2: IC3.95, SJ17.2
- removed net D57/ADC3: IC3.94, SJ18.2
- removed net D58/ADC4: IC3.93, SJ19.2
- removed net D59/ADC5: IC3.92, SJ20.2
- removed net D60/ADC6: IC3.91, SJ21.2
- removed net D61/ADC7: IC3.90, SJ22.2
- removed net D62/ADC8: IC3.89, SJ23.2
- removed net D63/ADC9: IC3.88, SJ24.2
- removed net D64/ADC10: IC3.87, SJ25.2
- removed net D65/ADC11: IC3.86, SJ26.2
- removed net D66/ADC12: IC3.85, SJ27.2
- removed net D68/ADC14: IC3.83, SJ31.2
- removed net D69/ADC15: IC3.82, SJ32.2
- removed net E-FAN: JP1.3, R35.2
- removed net E-FAN_CONTROL: JP4.3, SJ27.1
- removed net EDIR: JP3.7, U$7.CS/CCW
- removed net EDIR_CONTROL: JP2.7, SJ15.1
- removed net EENABLE: JP3.5, U$7.ENABLE
- removed net EENABLE_CONTROL: JP2.5, SJ13.1
- removed net ESTEP: JP3.6, U$7.CLK
- removed net ESTEP_CONTROL: JP2.6, SJ14.1
- removed net GND_CONTROL: C14.2, C28.1, C29.1, C30.1, C31.1, C36.1, C43.2, C44.C, C45.2, C47.C, C49.2, C5.2, C50.2, C51.C, C52.C, C6.2, C7.2, C8.2, IC1.8, IC2.1, IC3.11, IC3.32, IC3.62, IC3.81, IC3.99, IC5.2, IC5.3, IC5.4, ICSP.6, J3.GND, J3.GND2, JP4.12, JP4.9, L.C, ON.C, R67.1, R70.1, R71.1, RESET.1, RESET.2, SJ33.1, SJ33.2, SJ36.1, SJ36.2, U2.6, U2.GND1, U2.GND2, U6.18, U6.21, U6.25, U6.26, U6.7
- removed net HOTEND: JP1.2, R62.1
- removed net HOTEND_CONTROL: JP4.2, SJ26.1
- removed net N$35: SJ30.2
- removed net N$36: SJ29.2
- removed net PART-FAN: JP1.4, R28.2
- removed net PART-FAN_CONTROL: JP4.4, SJ28.1
- removed net TH1_HOTEND: C3.A, ETHERM.2, J1.10, JP1.8, R26.2
- removed net TH1_HOTEND_CONTROL: JP4.8, SJ32.1
- removed net TH2_BED: BEDTH.2, C4.A, JP1.7, R27.2
- removed net TH2_BED_CONTROL: JP4.7, SJ31.1
- removed net VM_CONTROL: JP4.10, SJ34.1
- removed net XDIR: JP3.16, U$17.CS/CCW
- removed net XDIR_CONTROL: JP2.16, SJ24.1
- removed net XENABLE: JP3.14, U$17.ENABLE
- removed net XENABLE_CONTROL: JP2.14, SJ22.1
- removed net XSTEP: JP3.15, U$17.CLK
- removed net XSTEP_CONTROL: JP2.15, SJ23.1
- removed net YDIR: JP3.13, U$1.CS/CCW
- removed net YDIR_CONTROL: JP2.13, SJ21.1
- removed net YENABLE: JP3.11, U$1.ENABLE
- removed net YENABLE_CONTROL: JP2.11, SJ19.1
- removed net YSTEP: JP3.12, U$1.CLK
- removed net YSTEP_CONTROL: JP2.12, SJ20.1
- removed net ZDIR: JP3.10, U$2.CS/CCW
- removed net ZDIR_CONTROL: JP2.10, SJ18.1
- removed net ZENABLE: JP3.8, U$2.ENABLE
- removed net ZENABLE_CONTROL: JP2.8, SJ16.1
- removed net ZSTEP: JP3.9, U$2.CLK
- removed net ZSTEP_CONTROL: JP2.9, SJ17.1
- removed net _E-ENDSTOP-C1_CONTROL: JP2.1, SJ9.1
- removed net _X-ENDSTOP-C1_CONTROL: JP2.4, SJ12.1
- removed net _Y-ENDSTOP-C1_CONTROL: JP2.3, SJ11.1
- removed net _Z-ENDSTOP-C1_CONTROL: JP2.2, SJ10.1
- new net D2/EENABLE: IC3.6, U$7.ENABLE
- new net D4/EDIR: IC3.1, U$7.CS/CCW
- new net D5/ESTEP: IC3.5, U$7.CLK
- new net D55/ADC1/ZENABLE: IC3.96, U$2.ENABLE
- new net D56/ADC2/ZSTEP: IC3.95, U$2.CLK
- new net D57/ADC3/ZDIR: IC3.94, U$2.CS/CCW
- new net D58/ADC4/YENABLE: IC3.93, U$1.ENABLE
- new net D59/ADC5/YSTEP: IC3.92, U$1.CLK
- new net D60/ADC6/YDIR: IC3.91, U$1.CS/CCW
- new net D61/ADC7/XENABLE: IC3.90, U$17.ENABLE
- new net D62/ADC8/XSTEP: IC3.89, U$17.CLK
- new net D63/ADC9/XDIR: IC3.88, U$17.CS/CCW
- new net D64/ADC10/BED: IC3.87, R24.1
- new net D65/ADC11/HOTEND: IC3.86, R62.1
- new net D66/ADC12/E-FAN: IC3.85, R35.2
- new net D68/ADC14/TH2_BED: BEDTH.2, C4.A, IC3.83, R27.2
- new net D69/ADC15/TH1_HOTEND: C3.A, ETHERM.2, IC3.82, J1.10, R26.2
- new net N$31: R74.2, U1.1
- new net N$32: R75.2, U1.3
- new net N$33: R76.2, U1.5
- new net N$34: R77.2, U1.7
- new net N$37: D20.A, U1.8
- new net N$38: D19.A, U1.6
- new net N$40: D17.A, U1.4
- new net N$42: D16.A, U1.2
- net 5VREG: now also C30.2, C51.A, C6.1, C7.1, C8.1, IC2.3, IC3.10, IC3.100, IC3.31, IC3.61, IC3.80, IC5.8, ICSP.2, JP6.1, L1.2, R60.1, R61.2, R64.2, R65.2, R74.1, R75.1, R76.1, R77.1, R78.2, R79.2, R80.2, R81.2, T2.2; no longer JP1.11
- net AGND: now also L3.1; no longer JP1.5
- net AVCC: now also L1.1; no longer JP1.6
- net D10: now also R81.1, U1.10; no longer SJ9.2
- net D3: now also R78.1, U1.16; no longer SJ12.2
- net D67/ADC13: now also R28.2; no longer SJ28.2
- net D8: now also R79.1, U1.14; no longer SJ11.2
- net D9: now also R80.1, U1.12; no longer SJ10.2
- net GND: now also C14.2, C28.1, C29.1, C30.1, C31.1, C36.1, C43.2, C44.C, C45.2, C47.C, C49.2, C5.2, C50.2, C51.C, C52.C, C6.2, C7.2, C8.2, IC1.8, IC2.1, IC3.11, IC3.32, IC3.62, IC3.81, IC3.99, IC5.2, IC5.3, IC5.4, ICSP.6, J3.GND, J3.GND2, L.C, L3.2, ON.C, R67.1, R70.1, R71.1, RESET.1, RESET.2, U1.11, U1.13, U1.15, U1.9, U2.6, U2.GND1, U2.GND2, U6.18, U6.21, U6.25, U6.26, U6.7; no longer JP1.12, JP1.9
- net VM: no longer JP1.10
- net VM_L2: no longer SJ34.2
- net _E-ENDSTOP-C1: now also D20.C; no longer JP3.1
- net _X-ENDSTOP-C1: now also D16.C; no longer JP3.4
- net _Y-ENDSTOP-C1: now also D17.C; no longer JP3.3
- net _Z-ENDSTOP-C1: now also D19.C; no longer JP3.2
Routing:
- net 5VREG: track 369.0 -> 514.5 mm, vias 9 -> 18
- net XENABLE: track 116.1 -> 0.00 mm, vias 1 -> 0
- net XSTEP: track 114.6 -> 0.00 mm, vias 1 -> 0
- net D62/ADC8/XSTEP: track 0.00 -> 110.3 mm, vias 0 -> 2
- net D61/ADC7/XENABLE: track 0.00 -> 110.0 mm, vias 0 -> 2
- net XDIR: track 109.4 -> 0.00 mm, vias 1 -> 0
- net D63/ADC9/XDIR: track 0.00 -> 107.2 mm, vias 0 -> 2
- net TH1_HOTEND: track 106.7 -> 0.00 mm, vias 2 -> 0
- net D69/ADC15/TH1_HOTEND: track 0.00 -> 104.9 mm, vias 0 -> 3
- net YENABLE: track 101.4 -> 0.00 mm, vias 1 -> 0
- net YSTEP: track 99.3 -> 0.00 mm, vias 1 -> 0
- net D68/ADC14/TH2_BED: track 0.00 -> 99.0 mm, vias 0 -> 2
- net TH2_BED: track 98.8 -> 0.00 mm, vias 1 -> 0
- net YDIR: track 94.1 -> 0.00 mm, vias 1 -> 0
- net D59/ADC5/YSTEP: track 0.00 -> 89.0 mm, vias 0 -> 2
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- added copper zone on layer 16, net D69/ADC15/TH1_HOTEND
- removed copper zone on layer 1, net GND
- removed copper zone on layer 16, net GND
- removed copper zone on layer 16, net TH1_HOTEND
Other:
- board size 210 x 100 mm -> 135 x 100 mm
- board text removed: "A-GND"
- board text removed: "A-VCC"
- board text removed: "E-DIR"
- board text removed: "E-EN"
- board text removed: "E-END"
- board text removed: "E-STP"
- board text removed: "TH1-HOTEND"
- board text removed: "TH2-BED"
- board text removed: "X-DIR"
- board text removed: "X-EN"
- board text removed: "X-END"
- board text removed: "X-STP"
- board text removed: "Y-DIR"
- board text removed: "Y-EN"
- board text removed: "Y-END"
- board text removed: "Y-STP"
- board text removed: "Z-DIR"
- board text removed: "Z-EN"
- board text removed: "Z-END"
- board text removed: "Z-STP"

Commit message: proto2
Parts:
- removed JP5, JP6: (no value), pinhead:1X01
- removed Q3: 16MHz, special:QS
- removed RESET: TS42, st-mod v1.4:TS42
- added D22: 5.1V, diode:SMB
- added Q4: 16Mhz, crystal:HC49UP
- added RST: MOMENTARY-SWITCH-SPST-PTH-6.0MM, SparkFun-Switches:TACTILE_SWITCH_PTH_6.0MM
- ON: device led:CHIP-LED0805 -> led:LED3MM
- moved R2 88.4 mm to (99.0, 31.0)
- moved LED6 88.4 mm to (99.0, 28.0)
- moved C52 46.7 mm to (106.9, 20.3), turned to 90 degrees
- moved ON 45.9 mm to (94.0, 28.0), flipped to the top
- moved R60 40.1 mm to (94.0, 31.0)
- moved IC2 39.2 mm to (100.9, 20.0), turned to 90 degrees
- moved R61 38.9 mm to (88.9, 29.4), turned to 90 degrees
- moved ICSP 33.8 mm to (125.2, 25.1), flipped to the top, turned to 270 degrees
- moved C51 32.6 mm to (94.3, 19.7), turned to 90 degrees
- moved C44 19.8 mm to (108.4, 10.7), turned to 270 degrees
- moved L 18.0 mm to (111.0, 56.0), turned to 0 degrees
- moved R77 14.7 mm to (96.9, 80.0)
- moved R55 13.7 mm to (111.0, 51.0), turned to 90 degrees
- moved R76 11.8 mm to (96.9, 77.0)
- moved R78 11.7 mm to (108.6, 71.4)
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Connections:
- removed net 5-GND: RESET.5
- removed net VM_L2: R66.2
- net 5VREG: now also D22.C; no longer JP6.1
- net GND: now also D22.A, ON.K, RST.3; no longer ON.C, RESET.1, RESET.2
- net RESET: now also RST.1; no longer RESET.3, RESET.4
- net VM: now also R66.2
- net V_USB: no longer JP5.1
- net XTAL1: now also Q4.1; no longer Q3.2
- net XTAL2: now also Q4.2; no longer Q3.1
Routing:
- net M8TXD: track 0.00 -> 78.2 mm
- net RESET: track 35.6 -> 112.3 mm, vias 0 -> 2
- net M8RXD: track 0.00 -> 74.9 mm, vias 0 -> 2
- net +3V3: track 34.5 -> 109.3 mm
- net VM: track 51.4 -> 96.2 mm, vias 4 -> 6
- net D51/MOSI: track 28.4 -> 69.0 mm, vias 1 -> 2
- net D50/MISO: track 48.4 -> 85.6 mm
- net D52/SCK: track 28.3 -> 65.2 mm, vias 1 -> 2
- net 5VREG: track 514.5 -> 546.7 mm, vias 18 -> 26
- net N$38: track 3.47 -> 18.6 mm, vias 0 -> 2
- net N$37: track 7.16 -> 20.7 mm, vias 0 -> 2
- net N$40: track 3.13 -> 16.7 mm, vias 0 -> 2
- net GND: track 43.7 -> 56.1 mm, vias 115 -> 220
- net D5/ESTEP: track 51.5 -> 42.3 mm
- net D61/ADC7/XENABLE: track 110.0 -> 100.9 mm
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- added copper zone on layer 1, net GND
- added copper zone on layer 16, net GND
Other:
- board size 135 x 100 mm -> 130 x 100 mm
- board text removed: "5V-REG"
- board text removed: "GND"
- board text removed: "VM"
