File: V3 Controller/MiniPrinterController.sch (EAGLE design)
At the start: 153 parts, among them IC9 XL1509-5.0E1, Q1 IRLR024, Q2 IRLR024, Q22 IRLR024, SW1 Legion SS21BBINPD Switch

Commit message: update
Parts:
- removed J5: (no value), SparkFun-Connectors:CONN_05X2SHD_LOCK
- removed SV1, SV2, SV3, SV4, SV5: (no value), con-lstb:MA04-1
- removed SV6: (no value), con-lstb:MA05-1
- removed SW1: Legion SS21BBINPD Switch, openbuilds-eagle-library:POWER-LEGION-SS21-SWITCH
- removed U$3, U$5: ATQ-FUSE, ATQ Fuse Holder out of 4.3mm pcb terminals:ATQ-FUSE
- removed X-END: Phoenix Pluggable 3.81mm 2 way, jt-con-phoenix-3.81:MC1.5/2
- added ETHERM: Phoenix Pluggable 3.81mm 2 way, jt-con-phoenix-3.81:MC1.5/2
- added J1, J2: (no value), SparkFun-Connectors:CONN_05X2SHD_LOCK
- added JP1: (no value), pinhead:PINHD-1X12
- added JP3: (no value), pinhead:PINHD-1X16
- LED6: device adafruit:LEDCHIPLED_0805 -> adafruit:LED3MM
Connections:
- removed net N$4: BED-2.1, U$3.P$2
- removed net PROBE: J8.9
- removed net V+FUSE: D14.C, SW1.L2, SW1.R2, U$4.P$2
- removed net VM-HOTEND: J5.4, J5.5, J5.6, U$5.P$2, X-END1G$2.1, X-END2G$2.1, X-END3G$2.1
- removed net X-END-C1: J7.9
- removed net Y-ENDSTOP-C1: J6.9
- removed net Z-ENDSTOP-C1: Z-CONN1.9
- new net N$40: JP1.9
- new net SPARE1: J2.10
- new net SPARE2: J2.9
- new net _E-ENDSTOP-C1: J7.9, JP3.1
- new net _X-ENDSTOP-C1: JP3.4, Z-CONN1.9
- new net _Y-ENDSTOP-C1: J6.9, JP3.3
- new net _Z-ENDSTOP-C1: J8.9, JP3.2
- net 5VREG: now also JP1.11
- net AGND: now also BEDTHG$1.1, ETHERMG$1.1, J1.9, JP1.5; no longer BEDTHG$2.1, J5.9, SV5.1
- net AVCC: now also JP1.6; no longer SV5.2
- net BED: now also JP1.1; no longer SV6.2
- net E-FAN: now also JP1.3; no longer SV6.3
- net E-FAN-NEG: now also J2.1, J2.2; no longer J5.7
- net EDIR: now also JP3.7; no longer SV4.4
- net EENABLE: now also JP3.5; no longer SV4.2
- net ESTEP: now also JP3.6; no longer SV4.3
- net GND: now also JP1.12; no longer SV1.1, SV2.1, SV3.1, SV4.1, SV6.1
- net HOTEND: now also JP1.2; no longer SV6.5
- net HOTEND-NEG1: now also J1.1, J1.2, J1.3, J1.4; no longer J5.1, J5.2, J5.3
- net PART-FAN: now also JP1.4; no longer SV6.4
- net PART-FAN-NEG: now also J2.5, J2.6; no longer J5.8
- net TH1_HOTEND: now also ETHERMG$2.1, J1.10, JP1.8; no longer J5.10, SV5.3
- net TH2_BED: now also BEDTHG$2.1, JP1.7; no longer BEDTHG$1.1, SV5.4
- net VM: now also BED-2.1, D14.C, J1.5, J1.6, J1.7, J1.8, J2.3, J2.4, J2.7, J2.8, JP1.10, U$4.P$2, X-END1G$2.1, X-END2G$2.1, X-END3G$2.1; no longer SW1.L1, SW1.R1, U$3.P$1, U$5.P$1
- net XDIR: now also JP3.16; no longer SV1.4
- net XENABLE: now also JP3.14; no longer SV1.2
- net XSTEP: now also JP3.15; no longer SV1.3
- net YDIR: now also JP3.13; no longer SV2.4
- net YENABLE: now also JP3.11; no longer SV2.2
- net YSTEP: now also JP3.12; no longer SV2.3
- net ZDIR: now also JP3.10; no longer SV3.4
- net ZENABLE: now also JP3.8; no longer SV3.2
- net ZSTEP: now also JP3.9; no longer SV3.3
Other:
- moved on the sheet: BEDTHG$1, BEDTHG$2

Commit message: update
Parts:
- added C14, C31, C36: 22p, SmartPrj:C-EU0603-RND
- added C28, C29, C5, C6, C7, C8: 100n, SmartPrj:C-EU0603-RND
- added C30: 100n, rcl:C-EUC0603
- added IC3: ATMEGA2560-16AU, atmel-2005:ATMEGA1280-16AU
- added IC5: LM358D, linear:LM358D
- added IC6: LP2985-33DBVR, texas:TPS77033
- added ICSP: ICSP, pinhead:PINHD-2X3
- added JP2: (no value), pinhead:PINHD-1X16
- added JP4: (no value), pinhead:PINHD-1X12
- added JP5, JP6: (no value), pinhead:PINHD-1X1
- added L: YELLOW, led:LEDCHIP-LED0805
- added ON: GREEN, led:LEDCHIP-LED0805
- added Q3: 16MHz, special:XTAL/S
- added R54: 27R, SmartPrj:R-EU_R0603
- added R55, R60, R68, R69: 1k, rcl:R-EU_R0603
- added R61, R64, R65, R66, R67: 10k, rcl:R-EU_R0603
- added RESET: TS42, st-mod v1.4:TS42
- added SJ10, SJ11, SJ12, SJ13, SJ14, SJ15, SJ16, SJ17, SJ18, SJ19, SJ20, SJ21, SJ22, SJ23, SJ24, SJ25, SJ26, SJ27, SJ28, SJ29, SJ30, SJ31, SJ32, SJ33, SJ34, SJ35, SJ36, SJ9: (no value), jumper:SJ
- added T2: FDN340P, zetex:PMOSSOT23
Connections:
- removed net N$40: JP1.9
- new net +3V3: C28.2, IC5B.-IN, IC6.OUT
- new net +5V: C30.2, C6.1, C7.1, C8.1, IC3.AVCC, IC3.VCC, IC3.VCC1, IC3.VCC2, IC3.VCC3, IC5P.V+, IC6.!EN, IC6.IN, ICSP.2, JP6.1, R60.1, R61.2, R64.2, R65.2, T2.S
- new net 5VREG_CONTROL: JP4.11, SJ35.1
- new net AGND_CONTROL: JP4.5, SJ29.1
- new net AREF: C5.1, IC3.AREF
- new net AVCC_CONTROL: JP4.6, SJ30.1
- new net BED_CONTROL: JP4.1, SJ25.1
- new net CMP: C29.2, IC5B.+IN, R66.1, R67.2
- new net D0: IC3.(RXD0/PCIN8)PE0, R68.2
- new net D1: IC3.(TXD0)PE1, R69.2
- new net D10: IC3.(OC2A/PCINT4)PB4, SJ9.2
- new net D11: IC3.(OC1A/PCINT5)PB5
- new net D12: IC3.(OC1B/PCINT6)PB6
- new net D13: IC3.(OC0A/OC1C/PCINT7)PB7, R55.1
- new net D14/TXD3: IC3.PJ1(TXD3/PCINT10)
- new net D15/RXD3: IC3.PJ0(RXD3/PCINT9)
- new net D16/TXD2: IC3.PH1(TXD2)
- new net D17/RXD2: IC3.PH0(RXD2)
- new net D18/TXD1: IC3.(TXD1/INT3)PD3
- new net D19/RXD1: IC3.(RXD1/INT2)PD2
- new net D2: IC3.(OC3B/INT4)PE4, SJ13.2
- new net D20/SDA: IC3.(SDA/INT1)PD1, R65.1
- new net D21/SCL: IC3.(SCL/INT0)PD0, R64.1
- new net D22: IC3.(AD0)PA0
- new net D23: IC3.(AD1)PA1
- new net D24: IC3.(AD2)PA2
- new net D25: IC3.(AD3)PA3
- new net D26: IC3.(AD4)PA4
- new net D27: IC3.(AD5)PA5
- new net D28: IC3.(AD6)PA6
- new net D29: IC3.(AD7)PA7
- new net D3: IC3.(OC3C/INT5)PE5, SJ12.2
- new net D30: IC3.(A15)PC7
- new net D31: IC3.(A14)PC6
- new net D32: IC3.(A13)PC5
- new net D33: IC3.(A12)PC4
- new net D34: IC3.(A11)PC3
- new net D35: IC3.(A10)PC2
- new net D36: IC3.(A9)PC1
- new net D37: IC3.(A8)PC0
- new net D38: IC3.(T0)PD7
- new net D39: IC3.(ALE)PG2
- new net D4: IC3.(OC0B)PG5, SJ15.2
- new net D40: IC3.(RD)PG1
- new net D41: IC3.(WR)PG0
- new net D42: IC3.PL7
- new net D43: IC3.PL6
- new net D44: IC3.PL5(OC5C)
- new net D45: IC3.PL4(OC5B)
- new net D46: IC3.PL3(OC5A)
- new net D47: IC3.PL2(T5)
- new net D48: IC3.PL1(ICP5)
- new net D49: IC3.PL0(ICP4)
- new net D5: IC3.(OC3A/AIN1)PE3, SJ14.2
- new net D50/MISO: IC3.(MISO/PCINT3)PB3, ICSP.1
- new net D51/MOSI: IC3.(MOSI/PCINT2)PB2, ICSP.4
- new net D52/SCK: IC3.(SCK/PCINT1)PB1, ICSP.3
- new net D53/SS: IC3.(SS/PCINT0)PB0
- new net D54/ADC0: IC3.(ADC0)PF0
- new net D55/ADC1: IC3.(ADC1)PF1, SJ16.2
- new net D56/ADC2: IC3.(ADC2)PF2, SJ17.2
- new net D57/ADC3: IC3.(ADC3)PF3, SJ18.2
- new net D58/ADC4: IC3.(ADC4/TCK)PF4, SJ19.2
- new net D59/ADC5: IC3.(ADC5/TMS)PF5, SJ20.2
- new net D60/ADC6: IC3.(ADC6/TDO)PF6, SJ21.2
- new net D61/ADC7: IC3.(ADC7/TDI)PF7, SJ22.2
- new net D62/ADC8: IC3.PK0(ADC8/PCINT16), SJ23.2
- new net D63/ADC9: IC3.PK1(ADC9/PCINT17), SJ24.2
- new net D64/ADC10: IC3.PK2(ADC10/PCINT18), SJ25.2
- new net D65/ADC11: IC3.PK3(ADC11/PCINT19), SJ26.2
- new net D66/ADC12: IC3.PK4(ADC12/PCINT20), SJ27.2
- new net D67/ADC13: IC3.PK5(ADC13/PCINT21), SJ28.2
- new net D68/ADC14: IC3.PK6(ADC14/PCINT22), SJ31.2
- new net D69/ADC15: IC3.PK7(ADC15/PCINT23), SJ32.2
- new net D8: IC3.PH5(OC4C), SJ11.2
- new net D9: IC3.PH6(OC2B), SJ10.2
- new net E-FAN_CONTROL: JP4.3, SJ27.1
- new net EDIR_CONTROL: JP2.7, SJ15.1
- new net EENABLE_CONTROL: JP2.5, SJ13.1
- new net ESTEP_CONTROL: JP2.6, SJ14.1
- new net GATE_CMD: IC5B.OUT, T2.G
- new net GND_CONTROL: C14.2, C28.1, C29.1, C30.1, C31.1, C36.1, C5.2, C6.2, C7.2, C8.2, IC3.AGND, IC3.GND, IC3.GND1, IC3.GND2, IC3.GND3, IC5A.+IN, IC5A.-IN, IC5P.V-, IC6.GND, ICSP.6, JP4.12, JP4.9, L.C, ON.C, R67.1, RESET.1, RESET.2, SJ33.1, SJ36.1
- new net HOTEND_CONTROL: JP4.2, SJ26.1
- new net M8RXD: R68.1
- new net M8TXD: R69.1
- new net N$13: ON.A, R60.2
- new net N$14: L.A, R55.2
- new net N$30: SJ35.2
- new net N$31: SJ34.2
- new net N$32: SJ33.2
- new net N$35: SJ30.2
- new net N$36: SJ29.2
- new net N$4: SJ36.2
- new net PART-FAN_CONTROL: JP4.4, SJ28.1
- new net PH3: IC3.PH3(OC4A)
- new net PH4: IC3.PH4(OC4B)
- new net RESET: C14.1, IC3.RESET, ICSP.5, R61.1, RESET.3, RESET.4
- new net TH1_HOTEND_CONTROL: JP4.8, SJ32.1
- new net TH2_BED_CONTROL: JP4.7, SJ31.1
- new net USBVCC: JP5.1, T2.D
- new net VIN: R66.2
- new net VM_CONTROL: JP4.10, SJ34.1
- new net XDIR_CONTROL: JP2.16, SJ24.1
- new net XENABLE_CONTROL: JP2.14, SJ22.1
- new net XSTEP_CONTROL: JP2.15, SJ23.1
- new net XTAL1: C31.2, Q3.2, R54.2
- new net XTAL1R: IC3.XTAL1, R54.1
- new net XTAL2: C36.2, IC3.XTAL2, Q3.1
- new net YDIR_CONTROL: JP2.13, SJ21.1
- new net YENABLE_CONTROL: JP2.11, SJ19.1
- new net YSTEP_CONTROL: JP2.12, SJ20.1
- new net ZDIR_CONTROL: JP2.10, SJ18.1
- new net ZENABLE_CONTROL: JP2.8, SJ16.1
- new net ZSTEP_CONTROL: JP2.9, SJ17.1
- new net _E-ENDSTOP-C1_CONTROL: JP2.1, SJ9.1
- new net _X-ENDSTOP-C1_CONTROL: JP2.4, SJ12.1
- new net _Y-ENDSTOP-C1_CONTROL: JP2.3, SJ11.1
- new net _Z-ENDSTOP-C1_CONTROL: JP2.2, SJ10.1
- net GND: now also JP1.9
Other:
- note added: "(MISO)"
- note added: "(MOSI)"
- note added: "(RX0)"
- note added: "(SCK)"
- note added: "(TX0)"
- note added: "0"
- note added: "1"
- note added: "14"
- note added: "15"
- note added: "16"
- note added: "17"
- note added: "18"
- note added: "19"
- note added: "2"
- note added: "20"
- note added: "21"
- note added: "3"
- note added: "4"
- note added: "5"
- note added: "6"
- note added: "7"
- note added: "pwm"
- note added: "serial in/out"

Commit message: update
Parts:
- removed IC6: LP2985-33DBVR, texas:TPS77033
- added C43, C45, C49, C50: 0.1uF, SparkFun:CAP0603-CAP
- added C44, C47, C51, C52: 10uF, SparkFun:CAP_POL1206
- added C46: 0.1uF, SmartPrj:C-EU0603-RND
- added D15: SS34, dp_devices:DIODE-DO-214AC
- added D21: RED/GRN BICOLOR 3528 LED, Wurth_Elektronik_Optoelectronics_rev15c:WL-SBTW-150141RB73100-R&B
- added IC1: 4050D, 40xx:4050D
- added IC2: 1117-33, v-reg:LD117AS33TR
- added J3: USB-C-Socket, SparkFun-Connectors:USB_C16PIN
- added R70, R71: 5.1k, SparkFun-Resistors:5.1KOHM5.1KOHM-0603-1/10W-1%
- added R72, R73: 1K, SparkFun:RESISTOR0603-RES
- added U2: USD-SOCKETUSD, SparkFun-Connectors_PETERMICROSDEBAY:USD-SOCKETUSD
- added U6: FT232RLSSOP, SparkFun:FT232RLSSOP
Connections:
- removed net N$31: SJ34.2
- removed net N$32: SJ33.2
- removed net USBVCC: JP5.1, T2.D
- removed net VIN: R66.2
- new net 3VUSB: C45.1, U6.3V3OUT
- new net CC1: J3.CC1, R71.2
- new net CC2: J3.CC2, R70.2
- new net CS: IC1A.O, U2.CS
- new net CTS: U6.CTS
- new net D+1: J3.D+, U6.USBDP
- new net D-1: J3.D-, U6.USBDM
- new net D6: IC3.(T3/INT6)PE6
- new net D7: IC3.(CLKO/ICP3/INT7)PE7
- new net DI: IC1B.O, U2.DI
- new net DTR: C46.1, U6.DTR
- new net RTS: U6.RTS
- new net RXLED: R72.1, U6.RXLED
- new net SC: IC1C.O, U2.SCK
- new net SHLD: J3.SHLD
- new net TXLED: R73.1, U6.TXLED
- new net VM_L2: R66.2, SJ34.2
- new net V_USB: C43.1, C44.+, D15.A, D21.A1, D21.A2, J3.VBUS, JP5.1, U6.VCC, U6.VCCIO
- new net V_USB_AFTERDIODE: D15.C, T2.D
- net +3V3: now also C47.+, C49.1, C50.1, C52.+, IC1P.VDD, IC2.OUT, U2.VCC; no longer IC6.OUT
- net +5V: now also C51.+, IC2.IN, SJ35.2; no longer IC6.!EN, IC6.IN
- net D50/MISO: now also U2.DO
- net D51/MOSI: now also IC1B.I
- net D52/SCK: now also IC1C.I
- net D53/SS: now also IC1A.I
- net GND_CONTROL: now also C43.2, C44.-, C45.2, C47.-, C49.2, C50.2, C51.-, C52.-, IC1P.VSS, IC2.ADJ, J3.GND, R70.1, R71.1, SJ33.2, SJ36.2, U2.GND, U2.SHIELD@3, U2.SHIELD@4, U6.AGND, U6.GND18, U6.GND21, U6.GND7, U6.TEST; no longer IC6.GND
- net M8RXD: now also U6.TXD
- net M8TXD: now also U6.RXD
- net N$30: now also D21.C1, R73.2; no longer SJ35.2
- net N$4: now also D21.C2, R72.2; no longer SJ36.2
- net RESET: now also C46.2
Other:
- note added: "USB TO SERIAL"

Commit message: update
Parts:
- removed JP1, JP4: (no value), pinhead:PINHD-1X12
- removed JP2, JP3: (no value), pinhead:PINHD-1X16
- removed SJ10, SJ11, SJ12, SJ13, SJ14, SJ15, SJ16, SJ17, SJ18, SJ19, SJ20, SJ21, SJ22, SJ23, SJ24, SJ25, SJ26, SJ27, SJ28, SJ29, SJ30, SJ31, SJ32, SJ33, SJ34, SJ35, SJ36, SJ9: (no value), jumper:SJ
- added D16, D17, D19, D20: M4, diode:DIODE-DO-214AC
- added L1, L3: 39nH, SparkFun:INDUCTOR0603
- added R74, R75, R76, R77: 1K, resistor:R-US_R0603
- added R78, R79, R80, R81: 10K, resistor:R-US_R0603
- added U1: TLP291-4, Toshiba TLP291-4 Optocoupler:TLP291-4
Connections:
- removed net +5V: C30.2, C51.+, C6.1, C7.1, C8.1, IC2.IN, IC3.AVCC, IC3.VCC, IC3.VCC1, IC3.VCC2, IC3.VCC3, IC5P.V+, ICSP.2, JP6.1, R60.1, R61.2, R64.2, R65.2, SJ35.2, T2.S
- removed net 5VREG_CONTROL: JP4.11, SJ35.1
- removed net AGND_CONTROL: JP4.5, SJ29.1
- removed net AVCC_CONTROL: JP4.6, SJ30.1
- removed net BED: JP1.1, R24.1
- removed net BED_CONTROL: JP4.1, SJ25.1
- removed net D2: IC3.(OC3B/INT4)PE4, SJ13.2
- removed net D4: IC3.(OC0B)PG5, SJ15.2
- removed net D5: IC3.(OC3A/AIN1)PE3, SJ14.2
- removed net D55/ADC1: IC3.(ADC1)PF1, SJ16.2
- removed net D56/ADC2: IC3.(ADC2)PF2, SJ17.2
- removed net D57/ADC3: IC3.(ADC3)PF3, SJ18.2
- removed net D58/ADC4: IC3.(ADC4/TCK)PF4, SJ19.2
- removed net D59/ADC5: IC3.(ADC5/TMS)PF5, SJ20.2
- removed net D60/ADC6: IC3.(ADC6/TDO)PF6, SJ21.2
- removed net D61/ADC7: IC3.(ADC7/TDI)PF7, SJ22.2
- removed net D62/ADC8: IC3.PK0(ADC8/PCINT16), SJ23.2
- removed net D63/ADC9: IC3.PK1(ADC9/PCINT17), SJ24.2
- removed net D64/ADC10: IC3.PK2(ADC10/PCINT18), SJ25.2
- removed net D65/ADC11: IC3.PK3(ADC11/PCINT19), SJ26.2
- removed net D66/ADC12: IC3.PK4(ADC12/PCINT20), SJ27.2
- removed net D68/ADC14: IC3.PK6(ADC14/PCINT22), SJ31.2
- removed net D69/ADC15: IC3.PK7(ADC15/PCINT23), SJ32.2
- removed net E-FAN: JP1.3, R35.2
- removed net E-FAN_CONTROL: JP4.3, SJ27.1
- removed net EDIR: JP3.7, U$7.CW/CCW
- removed net EDIR_CONTROL: JP2.7, SJ15.1
- removed net EENABLE: JP3.5, U$7.ENABLE
- removed net EENABLE_CONTROL: JP2.5, SJ13.1
- removed net ESTEP: JP3.6, U$7.CLK
- removed net ESTEP_CONTROL: JP2.6, SJ14.1
- removed net GND_CONTROL: C14.2, C28.1, C29.1, C30.1, C31.1, C36.1, C43.2, C44.-, C45.2, C47.-, C49.2, C5.2, C50.2, C51.-, C52.-, C6.2, C7.2, C8.2, IC1P.VSS, IC2.ADJ, IC3.AGND, IC3.GND, IC3.GND1, IC3.GND2, IC3.GND3, IC5A.+IN, IC5A.-IN, IC5P.V-, ICSP.6, J3.GND, JP4.12, JP4.9, L.C, ON.C, R67.1, R70.1, R71.1, RESET.1, RESET.2, SJ33.1, SJ33.2, SJ36.1, SJ36.2, U2.GND, U2.SHIELD@3, U2.SHIELD@4, U6.AGND, U6.GND18, U6.GND21, U6.GND7, U6.TEST
- removed net HOTEND: JP1.2, R62.1
- removed net HOTEND_CONTROL: JP4.2, SJ26.1
- removed net N$35: SJ30.2
- removed net N$36: SJ29.2
- removed net PART-FAN: JP1.4, R28.2
- removed net PART-FAN_CONTROL: JP4.4, SJ28.1
- removed net TH1_HOTEND: C3.+, ETHERMG$2.1, J1.10, JP1.8, R26.2
- removed net TH1_HOTEND_CONTROL: JP4.8, SJ32.1
- removed net TH2_BED: BEDTHG$2.1, C4.+, JP1.7, R27.2
- removed net TH2_BED_CONTROL: JP4.7, SJ31.1
- removed net VM_CONTROL: JP4.10, SJ34.1
- removed net XDIR: JP3.16, U$17.CW/CCW
- removed net XDIR_CONTROL: JP2.16, SJ24.1
- removed net XENABLE: JP3.14, U$17.ENABLE
- removed net XENABLE_CONTROL: JP2.14, SJ22.1
- removed net XSTEP: JP3.15, U$17.CLK
- removed net XSTEP_CONTROL: JP2.15, SJ23.1
- removed net YDIR: JP3.13, U$1.CW/CCW
- removed net YDIR_CONTROL: JP2.13, SJ21.1
- removed net YENABLE: JP3.11, U$1.ENABLE
- removed net YENABLE_CONTROL: JP2.11, SJ19.1
- removed net YSTEP: JP3.12, U$1.CLK
- removed net YSTEP_CONTROL: JP2.12, SJ20.1
- removed net ZDIR: JP3.10, U$2.CW/CCW
- removed net ZDIR_CONTROL: JP2.10, SJ18.1
- removed net ZENABLE: JP3.8, U$2.ENABLE
- removed net ZENABLE_CONTROL: JP2.8, SJ16.1
- removed net ZSTEP: JP3.9, U$2.CLK
- removed net ZSTEP_CONTROL: JP2.9, SJ17.1
- removed net _E-ENDSTOP-C1_CONTROL: JP2.1, SJ9.1
- removed net _X-ENDSTOP-C1_CONTROL: JP2.4, SJ12.1
- removed net _Y-ENDSTOP-C1_CONTROL: JP2.3, SJ11.1
- removed net _Z-ENDSTOP-C1_CONTROL: JP2.2, SJ10.1
- new net D2/EENABLE: IC3.(OC3B/INT4)PE4, U$7.ENABLE
- new net D4/EDIR: IC3.(OC0B)PG5, U$7.CW/CCW
- new net D5/ESTEP: IC3.(OC3A/AIN1)PE3, U$7.CLK
- new net D55/ADC1/ZENABLE: IC3.(ADC1)PF1, U$2.ENABLE
- new net D56/ADC2/ZSTEP: IC3.(ADC2)PF2, U$2.CLK
- new net D57/ADC3/ZDIR: IC3.(ADC3)PF3, U$2.CW/CCW
- new net D58/ADC4/YENABLE: IC3.(ADC4/TCK)PF4, U$1.ENABLE
- new net D59/ADC5/YSTEP: IC3.(ADC5/TMS)PF5, U$1.CLK
- new net D60/ADC6/YDIR: IC3.(ADC6/TDO)PF6, U$1.CW/CCW
- new net D61/ADC7/XENABLE: IC3.(ADC7/TDI)PF7, U$17.ENABLE
- new net D62/ADC8/XSTEP: IC3.PK0(ADC8/PCINT16), U$17.CLK
- new net D63/ADC9/XDIR: IC3.PK1(ADC9/PCINT17), U$17.CW/CCW
- new net D64/ADC10/BED: IC3.PK2(ADC10/PCINT18), R24.1
- new net D65/ADC11/HOTEND: IC3.PK3(ADC11/PCINT19), R62.1
- new net D66/ADC12/E-FAN: IC3.PK4(ADC12/PCINT20), R35.2
- new net D68/ADC14/TH2_BED: BEDTHG$2.1, C4.+, IC3.PK6(ADC14/PCINT22), R27.2
- new net D69/ADC15/TH1_HOTEND: C3.+, ETHERMG$2.1, IC3.PK7(ADC15/PCINT23), J1.10, R26.2
- new net N$31: R74.2, U1.1
- new net N$32: R75.2, U1.3
- new net N$33: R76.2, U1.5
- new net N$34: R77.2, U1.7
- new net N$37: D20.A, U1.8
- new net N$38: D19.A, U1.6
- new net N$40: D17.A, U1.4
- new net N$42: D16.A, U1.2
- net 5VREG: now also C30.2, C51.+, C6.1, C7.1, C8.1, IC2.IN, IC3.AVCC, IC3.VCC, IC3.VCC1, IC3.VCC2, IC3.VCC3, IC5P.V+, ICSP.2, JP6.1, L1.2, R60.1, R61.2, R64.2, R65.2, R74.1, R75.1, R76.1, R77.1, R78.2, R79.2, R80.2, R81.2, T2.S; no longer JP1.11
- net AGND: now also L3.1; no longer JP1.5
- net AVCC: now also L1.1; no longer JP1.6
- net D10: now also R81.1, U1.10; no longer SJ9.2
- net D3: now also R78.1, U1.16; no longer SJ12.2
- net D67/ADC13: now also R28.2; no longer SJ28.2
- net D8: now also R79.1, U1.14; no longer SJ11.2
- net D9: now also R80.1, U1.12; no longer SJ10.2
- net GND: now also C14.2, C28.1, C29.1, C30.1, C31.1, C36.1, C43.2, C44.-, C45.2, C47.-, C49.2, C5.2, C50.2, C51.-, C52.-, C6.2, C7.2, C8.2, IC1P.VSS, IC2.ADJ, IC3.AGND, IC3.GND, IC3.GND1, IC3.GND2, IC3.GND3, IC5A.+IN, IC5A.-IN, IC5P.V-, ICSP.6, J3.GND, L.C, L3.2, ON.C, R67.1, R70.1, R71.1, RESET.1, RESET.2, U1.11, U1.13, U1.15, U1.9, U2.GND, U2.SHIELD@3, U2.SHIELD@4, U6.AGND, U6.GND18, U6.GND21, U6.GND7, U6.TEST; no longer JP1.12, JP1.9
- net VM: no longer JP1.10
- net VM_L2: no longer SJ34.2
- net _E-ENDSTOP-C1: now also D20.C; no longer JP3.1
- net _X-ENDSTOP-C1: now also D16.C; no longer JP3.4
- net _Y-ENDSTOP-C1: now also D17.C; no longer JP3.3
- net _Z-ENDSTOP-C1: now also D19.C; no longer JP3.2
Other:
- note added: "TLP291-4"

Commit message: proto2
Parts:
- removed JP5, JP6: (no value), pinhead:PINHD-1X1
- removed Q3: 16MHz, special:XTAL/S
- removed RESET: TS42, st-mod v1.4:TS42
- added D22: 5.1V, diode:ZENER-DIODESMB
- added Q4: 16Mhz, crystal:CRYSTALHC49UP
- added RST: MOMENTARY-SWITCH-SPST-PTH-6.0MM, SparkFun-Switches:MOMENTARY-SWITCH-SPST-PTH-6.0MM
- ON: device led:LEDCHIP-LED0805 -> led:LED3MM
Connections:
- removed net VM_L2: R66.2
- net 5VREG: now also D22.C; no longer JP6.1
- net GND: now also D22.A, RST.2; no longer RESET.1, RESET.2
- net RESET: now also RST.1; no longer RESET.3, RESET.4
- net VM: now also R66.2
- net V_USB: no longer JP5.1
- net XTAL1: now also Q4.1; no longer Q3.2
- net XTAL2: now also Q4.2; no longer Q3.1
